Commit message: added maps and ekf

File: ros2_ws/src/abc_avc/avc_car/description/ros2_control/avc_car.ros2_control.xacro (robot description, xacro)
@@ -1,21 +1,23 @@
 <?xml version="1.0"?>
 <robot xmlns:xacro="http://www.ros.org/wiki/xacro">
-  <xacro:macro name="avc_car_ros2_control" params="name prefix">
-    <ros2_control name="${name}" type="system">
-      <hardware>
-        <plugin>avc_car/avc_carSystemHardware</plugin>
-        <param name="example_param_hw_start_duration_sec">0</param>
-        <param name="example_param_hw_stop_duration_sec">3.0</param>
-      </hardware>
-      <joint name="${prefix}virtual_front_wheel_joint">
-        <command_interface name="position"/>
-        <state_interface name="position"/>
-      </joint>
-      <joint name="${prefix}virtual_rear_wheel_joint">
-        <command_interface name="velocity"/>
-        <state_interface name="velocity"/>
-        <state_interface name="position"/>
-      </joint>
+    <ros2_control name="RobotControl" type="system">
+        <hardware>
+            <plugin>bicdrive_arduino/CarlikeBotSystemHardware</plugin>
+            <param name="front_wheel_name">virtual_front_wheel_joint</param> <!-- uhh TODO: might have to fix stuff with{prefix} if stuff is connected that way in the other urdf files-->
+            <param name="rear_wheel_name">virtual_rear_wheel_joint</param>
+            <param name="loop_rate">30</param>
+            <param name="device">/dev/serial/by-id/usb-1a86_USB2.0-Ser_-if00-port0</param>
+            <param name="baud_rate">9600</param>
+            <param name="timeout_ms">1000</param>
+        </hardware>
+        <joint name="virtual_front_wheel_joint">
+            <command_interface name="position"/>
+            <state_interface name="position"/>
+        </joint>
+        <joint name="virtual_rear_wheel_joint">
+            <command_interface name="velocity"/>
+            <state_interface name="velocity"/>
+            <state_interface name="position"/> <!-- (TODO: comment if we're NOT using joint_state_controller)-->
+        </joint>
     </ros2_control>
-  </xacro:macro>
 </robot>

Commit message: Things seem to work!
:3

File: ros2_ws/src/abc_avc/avc_car/description/ros2_control/avc_car.ros2_control.xacro (robot description, xacro)
@@ -1,23 +1,27 @@
 <?xml version="1.0"?>
 <robot xmlns:xacro="http://www.ros.org/wiki/xacro">
-    <ros2_control name="RobotControl" type="system">
-        <hardware>
-            <plugin>bicdrive_arduino/CarlikeBotSystemHardware</plugin>
-            <param name="front_wheel_name">virtual_front_wheel_joint</param> <!-- uhh TODO: might have to fix stuff with{prefix} if stuff is connected that way in the other urdf files-->
-            <param name="rear_wheel_name">virtual_rear_wheel_joint</param>
-            <param name="loop_rate">30</param>
-            <param name="device">/dev/serial/by-id/usb-1a86_USB2.0-Ser_-if00-port0</param>
-            <param name="baud_rate">9600</param>
-            <param name="timeout_ms">1000</param>
-        </hardware>
-        <joint name="virtual_front_wheel_joint">
-            <command_interface name="position"/>
-            <state_interface name="position"/>
-        </joint>
-        <joint name="virtual_rear_wheel_joint">
-            <command_interface name="velocity"/>
-            <state_interface name="velocity"/>
-            <state_interface name="position"/> <!-- (TODO: comment if we're NOT using joint_state_controller)-->
-        </joint>
+  <xacro:macro name="avc_car_ros2_control" params="name prefix">
+    <ros2_control name="${name}" type="system">
+      <hardware>
+        <plugin>avc_car/avc_carSystemHardware</plugin>
+        <param name="example_param_hw_start_duration_sec">0</param>
+        <param name="example_param_hw_stop_duration_sec">3.0</param>
+        <param name="loop_rate">69</param>
+        <param name="device">/dev/ttyACM0</param>
+        <param name="baud_rate">9600</param>
+        <param name="timeout_ms">1000</param>
+        <param name="traction_cal">0.00550369458</param>
+        <param name="steering_cal">1.0</param>
+      </hardware>
+      <joint name="${prefix}virtual_front_wheel_joint">
+        <command_interface name="position"/>
+        <state_interface name="position"/>
+      </joint>
+      <joint name="${prefix}virtual_rear_wheel_joint">
+        <command_interface name="velocity"/>
+        <state_interface name="velocity"/>
+        <state_interface name="position"/>
+      </joint>
     </ros2_control>
+  </xacro:macro>
 </robot>

Commit message: calibration and camera thing I think
idk lol

File: ros2_ws/src/abc_avc/avc_car/description/ros2_control/avc_car.ros2_control.xacro (robot description, xacro)
@@ -11,6 +11,8 @@
         <param name="baud_rate">9600</param>
         <param name="timeout_ms">1000</param>
-        <param name="traction_cal">0.00550369458</param>
+        <param name="traction_cal">3.961743677</param>
         <param name="steering_cal">1.0</param>
+        <param name="servo_vel">7.563093425</param>
+        <param name="servo_offset">90.0</param>
       </hardware>
       <joint name="${prefix}virtual_front_wheel_joint">

File: ros2_ws/src/abc_avc/avc_car/description/urdf/avc_car_description.urdf.xacro (robot description, xacro)
@@ -2,14 +2,14 @@
 <robot xmlns:xacro="http://www.ros.org/wiki/xacro">
   <xacro:macro name="avc_car" params="prefix">
-  <!-- Constants for robot dimensions -->
+  <!-- Constants for robot dimensions, everything has been changed except mass -->
   <xacro:property name="PI" value="3.1415926535897931"/>
   <xacro:property name="base_mass" value="4.0" /> <!-- arbitrary value for base mass -->
-  <xacro:property name="base_width" value="0.260" />
-  <xacro:property name="base_length" value="0.525" />
-  <xacro:property name="base_height" value="0.060" />
-  <xacro:property name="wheelbase" value="0.325" />
+  <xacro:property name="base_width" value="0.692" /><!-- side-to-side distance between wheels -->
+  <xacro:property name="base_length" value="0.872" /> <!-- length of car -->
+  <xacro:property name="base_height" value="0.2921" /> <!-- height of car -->
+  <xacro:property name="wheelbase" value="0.343" /> <!-- front-to-back distance between wheels -->
   <xacro:property name="wheel_mass" value="0.34055" /> <!-- arbitrary value for wheel mass -->
-  <xacro:property name="wheel_len" value="0.045" />
-  <xacro:property name="wheel_radius" value="0.05" />
+  <xacro:property name="wheel_len" value="0.07" /> <!-- thickness of wheel -->
+  <xacro:property name="wheel_radius" value="0.0685" /> <!-- radius of wheel -->
   <!-- <xacro:property name="wheeltrack" value="" -->
   <!-- Base Link -->

Commit message: Calibration implementation & fixes
Added code to make calibration values actually do things, adjusted calibration accordingly.
Still some cleanup to do, but this builds and runs correctly.

File: ros2_ws/src/abc_avc/avc_car/description/ros2_control/avc_car.ros2_control.xacro (robot description, xacro)
@@ -7,12 +7,13 @@
         <param name="example_param_hw_start_duration_sec">0</param>
         <param name="example_param_hw_stop_duration_sec">3.0</param>
-        <param name="loop_rate">69</param>
-        <param name="device">/dev/ttyACM0</param>
+        <param name="loop_rate">1000</param>
+        <param name="device">/dev/ttyACM1</param>
         <param name="baud_rate">9600</param>
-        <param name="timeout_ms">1000</param>
-        <param name="traction_cal">3.961743677</param>
-        <param name="steering_cal">1.0</param>
+        <param name="timeout_ms">150</param>
+        <param name="traction_cal">-12.7</param>
+        <param name="steering_cal">2.0</param>
         <param name="servo_vel">7.563093425</param>
-        <param name="servo_offset">90.0</param>
+        <param name="servo_offset">${pi/2}</param>
+        <param name="wheel_radius">0.0685</param>
       </hardware>
       <joint name="${prefix}virtual_front_wheel_joint">
@@ -25,4 +26,13 @@
         <state_interface name="position"/>
       </joint>
+      <!-- <sensor name="${prefix}fused_odom">
+        <state_interface name="position.x"/>
+        <state_interface name="position.y"/>
+        <state_interface name="position.z"/>
+        <state_interface name="orientation.x"/>
+        <state_interface name="orientation.y"/>
+        <state_interface name="orientation.z"/>
+        <state_interface name="orientation.w"/>
+      </sensor> -->
     </ros2_control>
   </xacro:macro>

File: ros2_ws/src/abc_avc/avc_car/description/urdf/avc_car_description.urdf.xacro (robot description, xacro)
@@ -5,7 +5,7 @@
   <xacro:property name="PI" value="3.1415926535897931"/>
   <xacro:property name="base_mass" value="4.0" /> <!-- arbitrary value for base mass -->
-  <xacro:property name="base_width" value="0.692" /><!-- side-to-side distance between wheels -->
-  <xacro:property name="base_length" value="0.872" /> <!-- length of car -->
-  <xacro:property name="base_height" value="0.2921" /> <!-- height of car -->
+  <xacro:property name="base_width" value="0.38" /><!-- side-to-side distance between wheels -->
+  <xacro:property name="base_length" value="0.56" /> <!-- length of car -->
+  <xacro:property name="base_height" value="0.20" /> <!-- height of car -->
   <xacro:property name="wheelbase" value="0.343" /> <!-- front-to-back distance between wheels -->
   <xacro:property name="wheel_mass" value="0.34055" /> <!-- arbitrary value for wheel mass -->

Commit message: meow

File: ros2_ws/src/abc_avc/avc_car/description/ros2_control/avc_car.ros2_control.xacro (robot description, xacro)
@@ -12,5 +12,5 @@
         <param name="timeout_ms">150</param>
         <param name="traction_cal">-12.7</param>
-        <param name="steering_cal">-2.0</param>
+        <param name="steering_cal">1.5</param>
         <param name="servo_vel">7.563093425</param>
         <param name="servo_offset">0</param>

File: ros2_ws/src/abc_avc/avc_car/description/urdf/avc_car_description.urdf.xacro (robot description, xacro)
@@ -17,4 +17,5 @@
   <link name="laser"/>
   <joint name="base_link_to_laser" type="fixed">
+    <origin xyz="0 0 0" rpy="0 0 ${PI}"/>
     <parent link="base_link"/>
     <child link="laser"/>
