Commit message: xacro and nav2_params from car

File: ros2_ws/src/abc_avc/avc_car/description/urdf/avc_car.materials.xacro (robot description, xacro)
@@ -17,4 +17,10 @@
     <color rgba="0.2 0.2 0.2 1.0"/>
   </material>
+  <material name="miku">
+    <color rgba="0.055 0.918 0.914 1.0"/>
+  </material>
+  <material name="pink">
+    <color rgba="0.94 0.05 0.537 1.0"/>
+  </material>
   <material name="orange">
     <color rgba="${255/255} ${108/255} ${10/255} 1.0"/>

File: ros2_ws/src/abc_avc/avc_car/description/urdf/avc_car_description.urdf.xacro (robot description, xacro)
@@ -22,17 +22,17 @@
   </joint>
   <!-- Front-->
-  <link name="front">
-      <visual>
-        <origin xyz="0 0 0" rpy="$0 0 0"/>
-        <geometry>
-          <box size="0.1 0.1 0.1"/>
-        </geometry>
-        <material name="blue"/>
-      </visual>
-  </link>
-    <joint name="base_to_front" type="fixed">
-      <parent link="base_link"/>
-      <child link="front"/>
-      <origin xyz="$0 0 ${base_height/2}" rpy="0 0 0"/>
+  <link name="${prefix}front_indicator">
+        <visual>
+          <origin xyz="${base_width/2} 0 ${base_height/2}" rpy="0 0 0"/>
+          <geometry>
+            <cylinder length="${wheel_len}" radius="${wheel_radius}"/>
+          </geometry>
+          <material name="pink"/>
+        </visual>
+    </link>
+    <joint name="${prefix}chassis_link_to_front_indicator" type="fixed">
+      <parent link="${prefix}chassis_link" />
+      <child link="${prefix}front_indicator" />
+      <origin xyz="0 0 0" rpy="0 0 0"/>
     </joint>
   <!-- Chassis -->
@@ -49,5 +49,5 @@
         <box size="${base_length} ${base_width} ${base_height}"/>
       </geometry>
-      <material name="orange"/>
+      <material name="miku"/>
     </visual>
     <inertial>
