Commit message: laser????????
AAAAAAAAAAAAAAAA

File: ros2_ws/src/abc_avc/avc_car/description/urdf/avc_car_description.urdf.xacro (robot description, xacro)
@@ -15,4 +15,9 @@
   <!-- Base Link -->
   <link name="${prefix}base_link" />
+  <link name="laser"/>
+  <joint name="base_link_to_laser" type="fixed">
+    <parent link="base_link"/>
+    <child link="laser"/>
+  </joint>
   <!-- Chassis -->
   <link name="${prefix}chassis_link">

Commit message: edited nav2 params, front indicator, twistmux

File: ros2_ws/src/abc_avc/avc_car/description/urdf/avc_car_description.urdf.xacro (robot description, xacro)
@@ -21,4 +21,19 @@
     <child link="laser"/>
   </joint>
+  <!-- Front-->
+  <link name="front">
+      <visual>
+        <origin xyz="0 0 0" rpy="$0 0 0"/>
+        <geometry>
+          <box size="0.1 0.1 0.1"/>
+        </geometry>
+        <material name="blue"/>
+      </visual>
+  </link>
+    <joint name="base_to_front" type="fixed">
+      <parent link="base_link"/>
+      <child link="front"/>
+      <origin xyz="$0 0 ${base_height/2}" rpy="0 0 0"/>
+    </joint>
   <!-- Chassis -->
   <link name="${prefix}chassis_link">

Commit message: misc changes
+miku

File: ros2_ws/src/abc_avc/avc_car/description/urdf/avc_car_description.urdf.xacro (robot description, xacro)
@@ -26,7 +26,7 @@
           <origin xyz="${base_width/2} 0 ${base_height/2}" rpy="0 0 0"/>
           <geometry>
-            <cylinder length="${wheel_len}" radius="${wheel_radius}"/>
+            <mesh filename="package://avc_car/meshes/reducedmiku.stl"/>
           </geometry>
-          <material name="pink"/>
+          <material name="miku"/>
         </visual>
     </link>
@@ -49,5 +49,5 @@
         <box size="${base_length} ${base_width} ${base_height}"/>
       </geometry>
-      <material name="miku"/>
+      <material name="blue"/>
     </visual>
     <inertial>

Commit message: Buckalization improvements for testing, sensor transforms

File: ros2_ws/src/abc_avc/avc_car/description/urdf/avc_car_description.urdf.xacro (robot description, xacro)
@@ -17,7 +17,25 @@
   <link name="laser"/>
   <joint name="base_link_to_laser" type="fixed">
-    <origin xyz="0 0 0" rpy="0 0 ${PI}"/>
+    <origin xyz="0.1 0 0.3" rpy="0 0 ${PI}"/>
     <parent link="base_link"/>
     <child link="laser"/>
+  </joint>
+  <link name="stereo_camera_center"/>
+  <joint name="base_link_to_stereo_center" type="fixed">
+    <origin xyz="0.2 0 0.22" rpy="0 0 0"/>
+    <parent link="base_link"/>
+    <child link="stereo_camera_center"/>
+  </joint>
+  <link name="camera_frame_left"/>
+  <joint name="stereo_center_to_left" type="fixed">
+    <origin xyz="0 0.128 0" rpy="0 0 0"/>
+    <parent link="stereo_camera_center"/>
+    <child link="camera_frame_left"/>
+  </joint>
+  <link name="camera_frame_right"/>
+  <joint name="stereo_center_to_left" type="fixed">
+    <origin xyz="0 -0.128 0" rpy="0 0 0"/>
+    <parent link="stereo_camera_center"/>
+    <child link="camera_frame_right"/>
   </joint>
   <!-- Front-->

Commit message: URDF fix real?
 also wow I keep getting confused between the repos

File: ros2_ws/src/abc_avc/avc_car/description/urdf/avc_car_description.urdf.xacro (robot description, xacro)
@@ -34,5 +34,5 @@
   </joint>
   <link name="camera_frame_right"/>
-  <joint name="stereo_center_to_left" type="fixed">
+  <joint name="stereo_center_to_right" type="fixed">
     <origin xyz="0 -0.128 0" rpy="0 0 0"/>
     <parent link="stereo_camera_center"/>
